File: Next4529.kicad_pcb (KiCad board)
At the start: 4 copper layers, 10.7 x 20.8 mm, 13 parts, among them U1 74LVC1G3157, U2 74LVC1G3157, U3 74LVC1G3157, U4 74LVC1G3157, U5 74LVC1G3157, U6 74LVC1G3157, U7 74LVC1G3157, U8 SLG46824V, U9 14529

Commit message: redesign
Parts:
- added U10: 74LVC1G66, Package_SON:Texas_USON-6_1x1.45mm_P0.5mm_SMD, F.Cu at (150.5, 88.9)
- added U8: 74LVC1G3157, Package_SON:Texas_USON-6_1x1.45mm_P0.5mm_SMD, F.Cu at (148.9, 88.9)
- added U9: 74LVC1G66, Package_SON:Texas_USON-6_1x1.45mm_P0.5mm_SMD, F.Cu at (150.5, 91.4)
- U1, U2, U3, U4, U5, U6, U7: footprint Package_TO_SOT_SMD:Vishay_PowerPAK_SC70-6L_Dual -> Package_SON:Texas_USON-6_1x1.45mm_P0.5mm_SMD
- moved U6 8.35 mm to (149.9, 79.9), turned to 180 degrees
- moved U5 5.82 mm to (146.9, 79.9)
- moved U4 4.75 mm to (149.9, 77.6)
- moved U3 4.33 mm to (149.9, 75.5)
- moved sda1 3.52 mm to (147.7, 86.3)
- moved U1 2.05 mm to (146.9, 75.6)
- moved U2 1.82 mm to (146.9, 77.7)
- moved U11 0.94 mm to (148.6, 83.4)
- moved C2 0.91 mm to (150.3, 81.1)
- moved U7 0.79 mm to (148.9, 91.4)
- moved scl1 0.67 mm to (149.3, 86.3)
- moved C1 0.18 mm to (146.6, 82.7), turned to 90 degrees
- renumbered U9 to IC1, U8 to U11
Connections:
- net /V renamed /ZC
- net Net-(U3-Pad4) renamed /Y01
- net Net-(U4-Pad4) renamed /Y23
- net Net-(U6-Pad4) renamed /Y
- U1 pad 4: Net-(U1-Pad4) -> /X01
- U11 pad 12: unconnected-(U8-IO7-Pad12) -> /WC
- U11 pad 13: unconnected-(U8-IO8-Pad13) -> /OE
- U11 pad 2: /YA -> /YC
- U11 pad 7: /YC -> /YA
- U2 pad 4: Net-(U2-Pad4) -> /X23
- U5 pad 1: Net-(U1-Pad4) -> /X23
- U5 pad 3: Net-(U2-Pad4) -> /X01
- U5 pad 4: /W -> /X
- U7 pad 1: /W -> /X
- U7 pad 4: /Z -> /ZG
Routing:
- net /X: track 0.00 -> 12.0 mm, vias 0 -> 2
- net Net-(U2-Pad4): track 12.0 -> 0.00 mm, vias 2 -> 0
- net /OE: track 0.00 -> 11.5 mm, vias 0 -> 3
- net Net-(U1-Pad4): track 11.0 -> 0.00 mm, vias 2 -> 0
- net GND: track 13.3 -> 2.40 mm, vias 24 -> 34
- net /Y: track 7.76 -> 16.6 mm
- net /W: track 9.86 -> 1.55 mm
- net /Y23: track 12.2 -> 4.17 mm, vias 2 -> 0
- net /X01: track 0.00 -> 7.06 mm
- net /WC: track 0.00 -> 6.23 mm, vias 0 -> 2
- net /YB: track 2.50 -> 7.81 mm, vias 1 -> 2
- net /sda: track 5.96 -> 1.65 mm
- net /Y3: track 5.09 -> 9.27 mm
- net /XC: track 4.40 -> 7.66 mm, vias 1 -> 2
- net /YC: track 7.19 -> 3.96 mm, vias 1 -> 2
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- added copper zone on In3.Cu, net +5V
- added copper zone on In2.Cu, net GND
- removed copper zone on In2.Cu, net +5V
- removed copper zone on In1.Cu, net GND
Other:
- copper layers 4 -> 6

Commit message: refine routing
Parts:
- added G***: LOGO, Library:BF-logo, B.Cu at (148.4, 90.6)
- added QR*****: https://github.com/jimbro1000/NX4529, Library:ProjectQR, B.Cu at (148.6, 75.5)
- U10, U9: value 74LVC1G66 -> 74LVC1G66DSF
Routing:
- net GND: track 2.40 -> 5.12 mm, vias 34 -> 32
- net /STx: track 9.50 -> 10.3 mm
- net /Y23: track 4.17 -> 4.32 mm, vias 0 -> 2
- net /X3: track 6.41 -> 6.48 mm, vias 0 -> 1
- net /Y2: vias 0 -> 1
- net /Y0: vias 0 -> 1
- net /X2: vias 0 -> 1
